Commit message: establish rtabmap control, nav2 control, added imu

File: description/urdf/palmvision.xacro (robot description, xacro)
@@ -1,25 +1,29 @@
 <?xml version="1.0"?>
-<robot xmlns:xacro="http://www.ros.org/wiki/xacro">
+<robot name='palmvision' xmlns:xacro="http://www.ros.org/wiki/xacro">
     <xacro:include filename='inertial_macros.xacro'/>
-    <xacro:property name='chassis_length' value='0.8'/>
-    <xacro:property name='chassis_width' value='0.5'/>
+    <xacro:property name='chassis_length' value='0.4'/>
+    <xacro:property name='chassis_width' value='0.3'/>
     <xacro:property name='chassis_height' value='0.15'/>
-    <xacro:property name='wheel_radius' value='0.1'/>
-    <xacro:property name='wheel_thickness' value='0.05'/>
+    <xacro:property name='wheel_radius' value='0.07'/>
+    <xacro:property name='wheel_thickness' value='0.04'/>
     <xacro:property name='component_length' value='0.15'/>
-    <xacro:property name='component_width' value='0.2'/>
-    <xacro:property name='component_height' value='0.2'/>
+    <xacro:property name='component_width' value='0.14'/>
+    <xacro:property name='component_height' value='0.1'/>
     <xacro:property name='camera_length' value='0.02'/>
     <xacro:property name='camera_width' value='0.02'/>
     <xacro:property name='camera_height' value='0.02'/>
+    <xacro:property name='imu_length' value='0.01'/>
+    <xacro:property name='imu_width' value='0.01'/>
+    <xacro:property name='imu_height' value='0.01'/>
     <xacro:property name='lidar_radius' value='0.075'/>
     <xacro:property name='lidar_thickness' value='0.065'/>
-    <xacro:property name='chassis_mass' value='20.0'/>
-    <xacro:property name='wheel_mass' value='3.0'/>
+    <xacro:property name='chassis_mass' value='4.0'/>
+    <xacro:property name='wheel_mass' value='2.0'/>
     <xacro:property name='component_mass' value='1.0'/>
     <xacro:property name='lidar_mass' value='0.23'/>
     <xacro:property name='camera_mass' value='0.55'/>
+    <xacro:property name='imu_mass' value='0.01'/>
     <xacro:property name='wheel_offset_x' value='${chassis_length/2 - wheel_radius}'/>
-    <xacro:property name='wheel_offset_y' value='${chassis_width/2 + wheel_thickness/2}'/>
+    <xacro:property name='wheel_offset_y' value='${chassis_width/2 + wheel_thickness/2 +0.01}'/>
     <xacro:property name='wheel_offset_z' value='-${chassis_height/2}'/>
     <material name="white">
@@ -115,4 +119,23 @@
         </collision>
     </link>
+    <link name="imu_link">
+        <xacro:inertial_box mass="${imu_mass}" x="${imu_length}" y="${imu_width}" z="${imu_height}">
+            <origin xyz="0 0 0" rpy="0 0 0"/>
+        </xacro:inertial_box>
+        <visual>
+            <origin xyz="0.0 0.0 0.0" rpy="0.0 0.0 0.0"/>
+            <geometry>
+                <box size="${imu_length} ${imu_width} ${imu_height}"/>
+            </geometry>
+            <material name="white"/>
+        </visual>
+        <collision>
+            <origin xyz="0.0 0.0 0.0" rpy="0.0 0.0 0.0"/>
+            <geometry>
+                <box size="${imu_length} ${imu_width} ${imu_height}"/>
+            </geometry>
+            <material name="white"/>
+        </collision>
+    </link>
     <link name="f_left_wheel_link">
         <visual>
@@ -124,5 +147,5 @@
         <collision>
             <geometry>
-                <cylinder radius="${wheel_radius}" length="${wheel_thickness}"/>
+                <sphere radius="${wheel_radius}"/>
             </geometry>
             <material name="blue"/>
@@ -141,5 +164,5 @@
         <collision>
             <geometry>
-                <cylinder radius="${wheel_radius}" length="${wheel_thickness}"/>
+                <sphere radius="${wheel_radius}"/>
             </geometry>
             <material name="blue"/>
@@ -158,5 +181,5 @@
         <collision>
             <geometry>
-                <cylinder radius="${wheel_radius}" length="${wheel_thickness}"/>
+                <sphere radius="${wheel_radius}"/>
             </geometry>
             <material name="blue"/>
@@ -175,5 +198,5 @@
         <collision>
             <geometry>
-                <cylinder radius="${wheel_radius}" length="${wheel_thickness}"/>
+                <sphere radius="${wheel_radius}"/>
             </geometry>
             <material name="blue"/>
@@ -189,5 +212,5 @@
     </joint>
     <joint name="chassis_joint" type="fixed">
-        <origin xyz="0.0 0.0 0.0" rpy="0.0 0.0 0.0"/>
+        <origin xyz="0.0 0.0 ${chassis_height}" rpy="0.0 0.0 0.0"/>
         <parent link="base_link"/>
         <child link="chassis_link"/>
@@ -204,7 +227,12 @@
     </joint>
     <joint name="camera_joint" type="fixed">
-        <origin xyz="${component_length/2 + camera_length/2} 0.0 0.08" rpy="0.0 0.0 0.0"/>
+        <origin xyz="${component_length/2 + camera_length/2} 0.0 0.0" rpy="0.0 0.0 0.0"/>
         <parent link="component_link"/>
         <child link="camera_link"/>
+    </joint>
+    <joint name="imu_joint" type="fixed">
+        <origin xyz="0.0 0.0 ${chassis_height/2 + imu_height/2}" rpy="0.0 0.0 0.0"/>
+        <parent link="chassis_link"/>
+        <child link="imu_link"/>
     </joint>
     <joint name="f_left_wheel_joint" type="continuous">
@@ -217,5 +245,5 @@
         <parent link="chassis_link"/>
         <child link="f_right_wheel_link"/>
-        <origin xyz="${wheel_offset_x} -${wheel_offset_y} ${wheel_offset_z}" rpy="-${pi/2} 0 0" />
+        <origin xyz="${wheel_offset_x} -${wheel_offset_y} ${wheel_offset_z}" rpy="${pi/2} 0 0" />
         <axis xyz="0 0 -1"/>
     </joint>
@@ -229,5 +257,5 @@
         <parent link="chassis_link"/>
         <child link="b_right_wheel_link"/>
-        <origin xyz="-${wheel_offset_x} -${wheel_offset_y} ${wheel_offset_z}" rpy="-${pi/2} 0 0" />
+        <origin xyz="-${wheel_offset_x} -${wheel_offset_y} ${wheel_offset_z}" rpy="${pi/2} 0 0" />
         <axis xyz="0 0 -1"/>
     </joint>

File: description/urdf/palmvision_gazebo.xacro (robot description, xacro)
@@ -41,5 +41,5 @@
         <plugin name="laser_controller" filename="libgazebo_ros_ray_sensor.so">
             <ros>
-                <remapping>~/out:=/cloud</remapping>
+                <remapping>~/out:=/lidar_points</remapping>
             </ros>
             <output_type>sensor_msgs/PointCloud2</output_type> <!-- Use PointCloud2 for 3D LiDAR -->
@@ -71,14 +71,29 @@
     </sensor>
 </gazebo>
+<gazebo reference="imu_link">
+  <sensor name="imu_sensor" type="imu">
+    <always_on>true</always_on>
+    <update_rate>100</update_rate>
+    <visualize>true</visualize>
+    <topic>__default_topic__</topic>
+    <plugin filename="libgazebo_ros_imu_sensor.so" name="imu_plugin">
+      <topicName>imu</topicName> <!-- Ensure this matches your UKF config -->
+      <bodyName>imu_link</bodyName>   <!-- This should be the same as the IMU link name -->
+      <updateRateHZ>100.0</updateRateHZ>
+      <gaussianNoise>0.0</gaussianNoise>
+      <xyzOffset>0 0 0</xyzOffset>
+      <rpyOffset>0 0 0</rpyOffset>
+      <frameName>imu</frameName> <!-- Frame name for TF broadcasts -->
+      <ros>
+        <remapping>~/out:=/imu</remapping> <!-- ROS 2 topic remapping -->
+      </ros>
+      <initialOrientationAsReference>false</initialOrientationAsReference>
+    </plugin>
+    <pose>0 0 0 0 0 0</pose>
+  </sensor>
+</gazebo>
 <gazebo reference="f_left_wheel_link">
   <mu1>0.9</mu1>
   <mu2>0.9</mu2>
-  <fdir1>1 0 0</fdir1>
-  <maxVel>0.0</maxVel>
-  <maxContacts>1</maxContacts>
-  <gravity>true</gravity>
-  <restitution_coefficient>1</restitution_coefficient>
-  <threshold>0</threshold>
-  <self_collide>1</self_collide>
   <material>Gazebo/Blue</material>
 </gazebo>
@@ -86,11 +101,4 @@
   <mu1>0.9</mu1>
   <mu2>0.9</mu2>
-  <fdir1>1 0 0</fdir1>
-  <maxVel>0.0</maxVel>
-  <maxContacts>1</maxContacts>
-  <gravity>true</gravity>
-  <restitution_coefficient>1</restitution_coefficient>
-  <threshold>0</threshold>
-  <self_collide>1</self_collide>
   <material>Gazebo/Blue</material>
 </gazebo>
@@ -98,11 +106,4 @@
   <mu1>0.9</mu1>
   <mu2>0.9</mu2>
-  <fdir1>1 0 0</fdir1>
-  <maxVel>0.0</maxVel>
-  <maxContacts>1</maxContacts>
-  <gravity>true</gravity>
-  <restitution_coefficient>1</restitution_coefficient>
-  <threshold>0</threshold>
-  <self_collide>1</self_collide>
   <material>Gazebo/Blue</material>
 </gazebo>
@@ -110,11 +111,4 @@
   <mu1>0.9</mu1>
   <mu2>0.9</mu2>
-  <fdir1>1 0 0</fdir1>
-  <maxVel>0.0</maxVel>
-  <maxContacts>1</maxContacts>
-  <gravity>true</gravity>
-  <restitution_coefficient>1</restitution_coefficient>
-  <threshold>0</threshold>
-  <self_collide>1</self_collide>
   <material>Gazebo/Blue</material>
 </gazebo>
