Commit message: Fixed Interface

File: description/urdf/palmvision.xacro (robot description, xacro)
@@ -2,186 +2,58 @@
 <robot name='palmvision' xmlns:xacro="http://www.ros.org/wiki/xacro">
     <xacro:include filename='inertial_macros.xacro'/>
+    <!-- COLORS -->
+    <material name="white">
+        <color rgba="1 1 1 1" />
+    </material>
+    <material name="orange">
+        <color rgba="1 0.3 0.1 1"/>
+    </material>
+    <material name="blue">
+        <color rgba="0.2 0.2 1 1"/>
+    </material>
+    <material name="black">
+        <color rgba="0 0 0 1"/>
+    </material>
+    <material name="red">
+        <color rgba="1 0 0 1"/>
+    </material>
+    <!-- CHASSIS PARAMS -->
     <xacro:property name='chassis_length' value='0.688'/>
     <xacro:property name='chassis_width' value='0.688'/>
     <xacro:property name='chassis_height' value='0.29'/>
-    <xacro:property name='wheel_radius' value='0.07'/>
-    <xacro:property name='wheel_thickness' value='0.04'/>
-    <xacro:property name='component_length' value='0.15'/>
-    <xacro:property name='component_width' value='0.14'/>
-    <xacro:property name='component_height' value='0.1'/>
+    <xacro:property name='chassis_mass' value='30.0'/>
+    <!-- WHEEL PARAMS -->
+    <xacro:property name='wheel_radius' value='0.127'/>
+    <xacro:property name='wheel_thickness' value='0.0762'/>
+    <xacro:property name='wheel_mass' value='2.0'/>
+    <xacro:property name='wheel_offset_x' value='${chassis_length/2 - wheel_radius/2}'/>
+    <xacro:property name='wheel_offset_y' value='${chassis_width/2 + wheel_thickness/2}'/>
+    <xacro:property name='wheel_offset_z' value='-${chassis_height/2}'/>
+    <!-- EXTENDED ARM PARAMS -->
+    <xacro:property name='arm_length' value='0.01'/>
+    <xacro:property name='arm_height' value='0.01'/>
+    <xacro:property name='arm_width' value='0.01'/>
+    <xacro:property name='arm_mass' value='0.2'/>
+    <xacro:property name='arm_offset_x' value='0'/>
+    <xacro:property name='arm_offset_y' value='${chassis_width/2 + arm_width/2}'/>
+    <xacro:property name='arm_offset_z' value='${chassis_height/2-arm_width}'/>
+    <!-- LIDAR PARAMS -->
+    <xacro:property name='lidar_radius' value='0.0379'/>
+    <xacro:property name='lidar_thickness' value='0.0347'/>
+    <xacro:property name='lidar_mass' value='0.2'/>
+    <xacro:property name='lidar_offset_x' value='${chassis_length/2 - lidar_radius}'/>
+    <xacro:property name='lidar_offset_y' value='0'/>
+    <xacro:property name='lidar_offset_z' value='${chassis_height/2 + lidar_thickness/2}'/>
+    <!-- CAMERA PARAMS -->
     <xacro:property name='camera_length' value='0.02'/>
     <xacro:property name='camera_width' value='0.02'/>
     <xacro:property name='camera_height' value='0.02'/>
-    <xacro:property name='lidar_radius' value='0.075'/>
-    <xacro:property name='lidar_thickness' value='0.065'/>
-    <xacro:property name='chassis_mass' value='4.0'/>
-    <xacro:property name='wheel_mass' value='2.0'/>
-    <xacro:property name='component_mass' value='1.0'/>
-    <xacro:property name='lidar_mass' value='0.23'/>
     <xacro:property name='camera_mass' value='0.55'/>
-    <xacro:property name='imu_mass' value='0.01'/>
-    <xacro:property name='wheel_offset_x' value='${chassis_length/2 - wheel_radius}'/>
-    <xacro:property name='wheel_offset_y' value='${chassis_width/2 + wheel_thickness/2 +0.01}'/>
-    <xacro:property name='wheel_offset_z' value='-${chassis_height/2}'/>
-    <material name="white">
-        <color rgba="1 1 1 1" />
-    </material>
-    <material name="orange">
-        <color rgba="1 0.3 0.1 1"/>
-    </material>
-    <material name="blue">
-        <color rgba="0.2 0.2 1 1"/>
-    </material>
-    <material name="black">
-        <color rgba="0 0 0 1"/>
-    </material>
-    <material name="red">
-        <color rgba="1 0 0 1"/>
-    </material>
+    <xacro:property name='camera_offset_x' value='${arm_length/2 + camera_length/2}'/>
+    <xacro:property name='camera_offset_y' value='0'/>
+    <xacro:property name='camera_offset_z' value='0'/>
     <!-- base -->
     <link name="base_link"></link>
     <link name="base_footprint"></link>
-    <link name="chassis_link">
-        <xacro:inertial_box mass="${chassis_mass}" x="${chassis_length}" y="${chassis_width}" z="${chassis_height}">
-            <origin xyz="0 0 0" rpy="0 0 0"/>
-        </xacro:inertial_box>
-        <visual>
-            <origin xyz="0.0 0.0 0.0" rpy="0.0 0.0 0.0"/>
-            <geometry>
-                <box size="${chassis_length} ${chassis_width} ${chassis_height}"/>
-            </geometry>
-            <material name="orange"/>
-        </visual>
-        <collision>
-            <origin xyz="0.0 0.0 0.0" rpy="0.0 0.0 0.0"/>
-            <geometry>
-                <box size="${chassis_length} ${chassis_width} ${chassis_height}"/>
-            </geometry>
-            <material name="orange"/>
-        </collision>
-    </link>
-    <link name="component_link">
-        <xacro:inertial_box mass="${component_mass}" x="${component_length}" y="${component_width}" z="${component_height}">
-            <origin xyz="0 0 0" rpy="0 0 0"/>
-        </xacro:inertial_box>
-        <visual>
-            <origin xyz="0.0 0.0 0.0" rpy="0.0 0.0 0.0"/>
-            <geometry>
-                <box size="${component_length} ${component_width} ${component_height}"/>
-            </geometry>
-            <material name="orange"/>
-        </visual>
-        <collision>
-            <origin xyz="0.0 0.0 0.0" rpy="0.0 0.0 0.0"/>
-            <geometry>
-                <box size="${component_length} ${component_width} ${component_height}"/>
-            </geometry>
-            <material name="orange"/>
-        </collision>
-    </link>
-    <link name="lidar_link">
-        <visual>
-            <geometry>
-                <cylinder radius="${lidar_radius}" length="${lidar_thickness}"/>
-            </geometry>
-            <material name="blue"/>
-        </visual>
-        <collision>
-            <geometry>
-                <cylinder radius="${lidar_radius}" length="${lidar_thickness}"/>
-            </geometry>
-            <material name="blue"/>
-        </collision>
-        <xacro:inertial_cylinder mass="${lidar_mass}" length="${lidar_thickness}" radius="${lidar_radius}">
-            <origin xyz="0 0 0" rpy="0 0 0"/>
-        </xacro:inertial_cylinder>
-    </link>
-    <link name="camera_link">
-        <xacro:inertial_box mass="${camera_mass}" x="${camera_length}" y="${camera_width}" z="${camera_height}">
-            <origin xyz="0 0 0" rpy="0 0 0"/>
-        </xacro:inertial_box>
-        <visual>
-            <origin xyz="0.0 0.0 0.0" rpy="0.0 0.0 0.0"/>
-            <geometry>
-                <box size="${camera_length} ${camera_width} ${camera_height}"/>
-            </geometry>
-            <material name="white"/>
-        </visual>
-        <collision>
-            <origin xyz="0.0 0.0 0.0" rpy="0.0 0.0 0.0"/>
-            <geometry>
-                <box size="${camera_length} ${camera_width} ${camera_height}"/>
-            </geometry>
-            <material name="white"/>
-        </collision>
-    </link>
-    <link name="f_left_wheel_link">
-        <visual>
-            <geometry>
-                <cylinder radius="${wheel_radius}" length="${wheel_thickness}"/>
-            </geometry>
-            <material name="blue"/>
-        </visual>
-        <collision>
-            <geometry>
-                <sphere radius="${wheel_radius}"/>
-            </geometry>
-            <material name="blue"/>
-        </collision>
-        <xacro:inertial_cylinder mass="${wheel_mass}" length="${wheel_thickness}" radius="${wheel_radius}">
-            <origin xyz="0 0 0" rpy="0 0 0"/>
-        </xacro:inertial_cylinder>
-    </link>
-    <link name="f_right_wheel_link">
-        <visual>
-            <geometry>
-                <cylinder radius="${wheel_radius}" length="${wheel_thickness}"/>
-            </geometry>
-            <material name="blue"/>
-        </visual>
-        <collision>
-            <geometry>
-                <sphere radius="${wheel_radius}"/>
-            </geometry>
-            <material name="blue"/>
-        </collision>
-        <xacro:inertial_cylinder mass="${wheel_mass}" length="${wheel_thickness}" radius="${wheel_radius}">
-            <origin xyz="0 0 0" rpy="0 0 0"/>
-        </xacro:inertial_cylinder>
-    </link>
-    <link name="b_left_wheel_link">
-        <visual>
-            <geometry>
-                <cylinder radius="${wheel_radius}" length="${wheel_thickness}"/>
-            </geometry>
-            <material name="blue"/>
-        </visual>
-        <collision>
-            <geometry>
-                <sphere radius="${wheel_radius}"/>
-            </geometry>
-            <material name="blue"/>
-        </collision>
-        <xacro:inertial_cylinder mass="${wheel_mass}" length="${wheel_thickness}" radius="${wheel_radius}">
-            <origin xyz="0 0 0" rpy="0 0 0"/>
-        </xacro:inertial_cylinder>
-    </link>
-    <link name="b_right_wheel_link">
-        <visual>
-            <geometry>
-                <cylinder radius="${wheel_radius}" length="${wheel_thickness}"/>
-            </geometry>
-            <material name="blue"/>
-        </visual>
-        <collision>
-            <geometry>
-                <sphere radius="${wheel_radius}"/>
-            </geometry>
-            <material name="blue"/>
-        </collision>
-        <xacro:inertial_cylinder mass="${wheel_mass}" length="${wheel_thickness}" radius="${wheel_radius}">
-            <origin xyz="0 0 0" rpy="0 0 0"/>
-        </xacro:inertial_cylinder>
-    </link>
     <joint name="base_footprint_joint" type="fixed">
         <origin xyz="0.0 0.0 0.0" rpy="0.0 0.0 0.0"/>
@@ -189,4 +61,23 @@
         <child link="base_footprint"/>
     </joint>
+    <link name="chassis_link">
+        <xacro:inertial_box mass="${chassis_mass}" x="${chassis_length}" y="${chassis_width}" z="${chassis_height}">
+            <origin xyz="0 0 0" rpy="0 0 0"/>
+        </xacro:inertial_box>
+        <visual>
+            <origin xyz="0.0 0.0 0.0" rpy="0.0 0.0 0.0"/>
+            <geometry>
+                <box size="${chassis_length} ${chassis_width} ${chassis_height}"/>
+            </geometry>
+            <material name="orange"/>
+        </visual>
+        <collision>
+            <origin xyz="0.0 0.0 0.0" rpy="0.0 0.0 0.0"/>
+            <geometry>
+                <box size="${chassis_length} ${chassis_width} ${chassis_height}"/>
+            </geometry>
+            <material name="orange"/>
+        </collision>
+    </link>
     <joint name="chassis_joint" type="fixed">
         <origin xyz="0.0 0.0 ${chassis_height}" rpy="0.0 0.0 0.0"/>
@@ -194,19 +85,144 @@
         <child link="chassis_link"/>
     </joint>
-    <joint name="component_joint" type="fixed">
-        <origin xyz="-${chassis_length/2 - component_length/2} 0.0 ${chassis_height/2 + component_height/2}" rpy="0.0 0.0 0.0"/>
-        <parent link="chassis_link"/>
-        <child link="component_link"/>
-    </joint>
+    <link name="arm_link">
+        <xacro:inertial_box mass="${arm_mass}" x="${arm_length}" y="${arm_width}" z="${arm_height}">
+            <origin xyz="0 0 0" rpy="0 0 0"/>
+        </xacro:inertial_box>
+        <visual>
+            <origin xyz="0.0 0.0 0.0" rpy="0.0 0.0 0.0"/>
+            <geometry>
+                <box size="${arm_length} ${arm_width} ${arm_height}"/>
+            </geometry>
+            <material name="orange"/>
+        </visual>
+        <collision>
+            <origin xyz="0.0 0.0 0.0" rpy="0.0 0.0 0.0"/>
+            <geometry>
+                <box size="${arm_length} ${arm_width} ${arm_height}"/>
+            </geometry>
+            <material name="orange"/>
+        </collision>
+    </link>
+    <joint name="arm_joint" type="revolute">
+        <origin xyz="${arm_offset_x} ${arm_offset_y} ${arm_offset_z}" rpy="0.0 0.0 ${pi/2}"/>
+        <parent link="chassis_link"/>
+        <child link="arm_link"/>
+        <axis xyz="0.0 1.0 0.0"/>
+        <limit lower="${-pi/2}" upper="${pi/2}" effort="10.0" velocity="2.0"/>
+    </joint>
+    <link name="camera_link">
+        <xacro:inertial_box mass="${camera_mass}" x="${camera_length}" y="${camera_width}" z="${camera_height}">
+            <origin xyz="0 0 0" rpy="0 0 0"/>
+        </xacro:inertial_box>
+        <visual>
+            <origin xyz="0.0 0.0 0.0" rpy="0.0 0.0 0.0"/>
+            <geometry>
+                <box size="${camera_length} ${camera_width} ${camera_height}"/>
+            </geometry>
+            <material name="white"/>
+        </visual>
+        <collision>
+            <origin xyz="0.0 0.0 0.0" rpy="0.0 0.0 0.0"/>
+            <geometry>
+                <box size="${camera_length} ${camera_width} ${camera_height}"/>
+            </geometry>
+            <material name="white"/>
+        </collision>
+    </link>
+    <joint name="camera_joint" type="fixed">
+        <origin xyz="${camera_offset_x} ${camera_offset_y} ${camera_offset_z}" rpy="0.0 0.0 0.0"/>
+        <parent link="arm_link"/>
+        <child link="camera_link"/>
+    </joint>
+    <link name="lidar_link">
+        <visual>
+            <geometry>
+                <cylinder radius="${lidar_radius}" length="${lidar_thickness}"/>
+            </geometry>
+            <material name="blue"/>
+        </visual>
+        <collision>
+            <geometry>
+                <cylinder radius="${lidar_radius}" length="${lidar_thickness}"/>
+            </geometry>
+            <material name="blue"/>
+        </collision>
+        <xacro:inertial_cylinder mass="${lidar_mass}" length="${lidar_thickness}" radius="${lidar_radius}">
+            <origin xyz="0 0 0" rpy="0 0 0"/>
+        </xacro:inertial_cylinder>
+    </link>
     <joint name="lidar_joint" type="fixed">
-        <origin xyz="0.0 0.0 ${component_height/2 + lidar_thickness/2}" rpy="0.0 0.0 0.0"/>
-        <parent link="component_link"/>
+        <origin xyz="${lidar_offset_x} ${lidar_offset_y} ${lidar_offset_z}" rpy="0.0 0.0 0.0"/>
+        <parent link="chassis_link"/>
         <child link="lidar_link"/>
     </joint>
-    <joint name="camera_joint" type="fixed">
-        <origin xyz="${component_length/2 + camera_length/2} 0.0 0.0" rpy="0.0 0.0 0.0"/>
-        <parent link="component_link"/>
-        <child link="camera_link"/>
-    </joint>
+    <link name="f_left_wheel_link">
+        <visual>
+            <geometry>
+                <cylinder radius="${wheel_radius}" length="${wheel_thickness}"/>
+            </geometry>
+            <material name="blue"/>
+        </visual>
+        <collision>
+            <geometry>
+                <cylinder radius="${wheel_radius}" length="${wheel_thickness}"/>
+            </geometry>
+            <material name="blue"/>
+        </collision>
+        <xacro:inertial_cylinder mass="${wheel_mass}" length="${wheel_thickness}" radius="${wheel_radius}">
+            <origin xyz="0 0 0" rpy="0 0 0"/>
+        </xacro:inertial_cylinder>
+    </link>
+    <link name="f_right_wheel_link">
+        <visual>
+            <geometry>
+                <cylinder radius="${wheel_radius}" length="${wheel_thickness}"/>
+            </geometry>
+            <material name="blue"/>
+        </visual>
+        <collision>
+            <geometry>
+                <cylinder radius="${wheel_radius}" length="${wheel_thickness}"/>
+            </geometry>
+            <material name="blue"/>
+        </collision>
+        <xacro:inertial_cylinder mass="${wheel_mass}" length="${wheel_thickness}" radius="${wheel_radius}">
+            <origin xyz="0 0 0" rpy="0 0 0"/>
+        </xacro:inertial_cylinder>
+    </link>
+    <link name="b_left_wheel_link">
+        <visual>
+            <geometry>
+                <cylinder radius="${wheel_radius}" length="${wheel_thickness}"/>
+            </geometry>
+            <material name="blue"/>
+        </visual>
+        <collision>
+            <geometry>
+                <cylinder radius="${wheel_radius}" length="${wheel_thickness}"/>
+            </geometry>
+            <material name="blue"/>
+        </collision>
+        <xacro:inertial_cylinder mass="${wheel_mass}" length="${wheel_thickness}" radius="${wheel_radius}">
+            <origin xyz="0 0 0" rpy="0 0 0"/>
+        </xacro:inertial_cylinder>
+    </link>
+    <link name="b_right_wheel_link">
+        <visual>
+            <geometry>
+                <cylinder radius="${wheel_radius}" length="${wheel_thickness}"/>
+            </geometry>
+            <material name="blue"/>
+        </visual>
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
File: description/urdf/palmvision_gazebo.xacro (robot description, xacro)
@@ -3,14 +3,4 @@
 <gazebo reference="chassis_link">
   <material>Gazebo/Orange</material>
-  <mu1>0.2</mu1>
-  <mu2>0.2</mu2>
-  <self_collide>true</self_collide>
-  <gravity>true</gravity>
-</gazebo>
-<gazebo reference="component_link">
-  <material>Gazebo/Orange</material>
-  <mu1>0.2</mu1>
-  <mu2>0.2</mu2>
-  <self_collide>true</self_collide>
   <gravity>true</gravity>
 </gazebo>
@@ -28,13 +18,8 @@
                     <max_angle>3.14</max_angle>
                 </horizontal>
-                <vertical>
-                    <samples>16</samples> <!-- Number of vertical layers -->
-                    <min_angle>-0.0</min_angle> <!-- Minimum vertical angle (in radians, ~-15 degrees) -->
-                    <max_angle>0.2618</max_angle> <!-- Maximum vertical angle (in radians, ~15 degrees) -->
-                </vertical>
             </scan>
             <range>
                 <min>0.3</min>
-                <max>10</max>
+                <max>15</max>
             </range>
         </ray>
@@ -113,4 +98,6 @@
   <material>Gazebo/Blue</material>
 </gazebo>
-<!-- lidar -->
+<gazebo reference="arm_link">
+  <material>Gazebo/Blue</material>
+</gazebo>
 </robot>

File: description/urdf/ros2_control.xacro (robot description, xacro)
@@ -37,4 +37,8 @@
             <state_interface name="position"/>
         </joint>
+        <joint name="arm_joint">
+            <command_interface name="position"/>
+            <state_interface name="position"/>
+        </joint>
     </ros2_control>
     <gazebo>

File: palmvision_control/description/ros2_control/ros2_control.xacro (robot description, xacro)
@@ -8,14 +8,9 @@
             <param name="back_left_wheel_name">b_left_wheel_joint</param>
             <param name="back_right_wheel_name">b_right_wheel_joint</param>
-            <param name="servo name">arm_joint</param>
-            <param name="loop_rate">30</param>
-            <param name="device">/tty/ACM0</param>
-            <param name="baud_rate">57600</param>
+            <param name="servo_name">arm_joint</param>
+            <param name="device">/dev/ttyUSB0</param>
+            <param name="baud_rate">115200</param>
             <param name="timeout_ms">1000</param>
-            <param name="enc_counts_per_rev">120</param>
-            <param name="pid_p">20</param>
-            <param name="pid_d">12</param>
-            <param name="pid_i">0</param>
-            <param name="pid_o">50</param>
+            <param name="enc_counts_per_rev">480</param>
         </hardware>
         <joint name="f_left_wheel_joint">

File: palmvision_control/description/urdf/palmrobot.xacro (robot description, xacro)
@@ -35,6 +35,6 @@
     <xacro:property name='arm_width' value='0.01'/>
     <xacro:property name='arm_mass' value='0.2'/>
-    <xacro:property name='arm_offset_x' value='${chassis_length/2 + arm_height/2}'/>
-    <xacro:property name='arm_offset_y' value='0'/>
+    <xacro:property name='arm_offset_x' value='0'/>
+    <xacro:property name='arm_offset_y' value='${chassis_width/2 + arm_width/2}'/>
     <xacro:property name='arm_offset_z' value='${chassis_height/2-arm_width}'/>
     <!-- LIDAR PARAMS -->
@@ -105,5 +105,5 @@
     </link>
     <joint name="arm_joint" type="revolute">
-        <origin xyz="${arm_offset_x} ${arm_offset_y} ${arm_offset_z}" rpy="0.0 0.0 0.0"/>
+        <origin xyz="${arm_offset_x} ${arm_offset_y} ${arm_offset_z}" rpy="0.0 0.0 ${pi/2}"/>
         <parent link="chassis_link"/>
         <child link="arm_link"/>
