Commit message: Fixed Interface

File: palmvision_control/description/urdf/palmrobot.xacro (robot description, xacro)
@@ -135,4 +135,26 @@
         <child link="camera_link"/>
     </joint>
+    <link name="support_link">
+        <visual>
+            <geometry>
+                <cylinder radius="0.01" length="0.15"/>
+            </geometry>
+            <material name="blue"/>
+        </visual>
+        <collision>
+            <geometry>
+                <cylinder radius="0.01" length="0.15"/>
+            </geometry>
+            <material name="blue"/>
+        </collision>
+        <xacro:inertial_cylinder mass="0.2" length="0.01" radius="0.15">
+            <origin xyz="0 0 0" rpy="0 0 0"/>
+        </xacro:inertial_cylinder>
+    </link>
+    <joint name="support_joint" type="fixed">
+        <origin xyz="${lidar_offset_x} ${lidar_offset_y} ${lidar_offset_z}" rpy="0.0 0.0 0.0"/>
+        <parent link="chassis_link"/>
+        <child link="support_link"/>
+    </joint>
     <link name="lidar_link">
         <visual>
@@ -153,6 +175,6 @@
     </link>
     <joint name="lidar_joint" type="fixed">
-        <origin xyz="${lidar_offset_x} ${lidar_offset_y} ${lidar_offset_z}" rpy="0.0 0.0 0.0"/>
-        <parent link="chassis_link"/>
+        <origin xyz="0 0 ${0.15/2 + lidar_thickness/2}" rpy="0.0 0.0 0.0"/>
+        <parent link="support_link"/>
         <child link="lidar_link"/>
     </joint>
