Commit message: Fixed esp32 and ydlidar udev rules, writing for cam control node -- Not Done

File: palmvision_control/description/ros2_control/ros2_control.xacro (robot description, xacro)
@@ -9,5 +9,5 @@
             <param name="back_right_wheel_name">b_right_wheel_joint</param>
             <param name="servo_name">arm_joint</param>
-            <param name="device">/dev/ttyUSB0</param>
+            <param name="device">/dev/esp32</param>
             <param name="baud_rate">115200</param>
             <param name="timeout_ms">1000</param>

File: palmvision_control/description/urdf/palmrobot.xacro (robot description, xacro)
@@ -174,4 +174,21 @@
         </xacro:inertial_cylinder>
     </link>
+    <link name="pseudo_lidar_link">
+        <visual>
+            <geometry>
+                <cylinder radius="${lidar_radius}" length="${lidar_thickness}"/>
+            </geometry>
+            <material name="blue"/>
+        </visual>
+        <collision>
+            <geometry>
+                <cylinder radius="${lidar_radius}" length="${lidar_thickness}"/>
+            </geometry>
+            <material name="blue"/>
+        </collision>
+        <xacro:inertial_cylinder mass="${lidar_mass}" length="${lidar_thickness}" radius="${lidar_radius}">
+            <origin xyz="0 0 0" rpy="0 0 0"/>
+        </xacro:inertial_cylinder>
+    </link>
     <joint name="lidar_joint" type="fixed">
         <origin xyz="0 0 ${0.15/2 + lidar_thickness/2}" rpy="0.0 0.0 0.0"/>
@@ -179,4 +196,9 @@
         <child link="lidar_link"/>
     </joint>
+    <joint name="pseudo_lidar_joint" type="fixed">
+        <origin xyz="0 0 ${0.15/2 + lidar_thickness/2}" rpy="0.0 0.0 0.0"/>
+        <parent link="support_link"/>
+        <child link="pseudo_lidar_link"/>
+    </joint>
     <link name="f_left_wheel_link">
         <visual>
